File: KiCad/Ionosonde_watchdog/Ionosonde_watchdog.sch (KiCad schematic (older format))
At the start: 42 parts

Commit message: New schematics
Parts:
- removed D? (x3): LED, symbol Device:LED
- removed J?: INTERLOCKpin, symbol Connector_Generic:Conn_01x01
- removed J?: SERVERFAILpin, symbol Connector_Generic:Conn_01x01
- removed J?: TXONpin, symbol Connector_Generic:Conn_01x01
- removed J?: RELAYpin, symbol Connector_Generic:Conn_01x01
- removed J?: USRPpin, symbol Connector_Generic:Conn_01x01
- removed J?: NTCpin, symbol Connector_Generic:Conn_01x01
- removed J?: ONE_WIRE_BUS, symbol Connector_Generic:Conn_01x01
- removed J?: GND, symbol Connector_Generic:Conn_01x01
- removed J?: 5V, symbol Connector_Generic:Conn_01x01
- removed J?: WATCHDOGpin, symbol Connector_Generic:Conn_01x01
- removed J?: Screw_Terminal_01x02, symbol Connector:Screw_Terminal_01x02
- removed J?: RESET, symbol Connector_Generic:Conn_01x01
- removed K?: SILxx-1Cxx-51x, Relay_THT:Relay_SPDT_StandexMeder_SIL_Form1C, symbol Relay:SILxx-1Cxx-51x
- removed Q?: TIP121, Package_TO_SOT_THT:TO-220-3_Vertical, symbol Transistor_BJT:TIP121
- removed R? (x2): 270, symbol Device:R
- removed U?: MAX693, symbol Ionosonde_watchdog:MAX693
- added C3: 3n3, symbol Device:C
- added C4, C5: 100n, symbol Device:C
- added D1: GREEN LED, symbol Device:LED
- added D2, D5: RED LED, symbol Device:LED
- added R1, R7: 270, symbol Device:R
- added R12, R9: 47k, symbol Device:R
- added SW1: SW_DPDT_x2, symbol Switch:SW_DPDT_x2
- added SW3: SW_SPDT, symbol Switch:SW_SPDT
- added U3: PVN012, symbol pvn012:PVN012
- added U4: UCC2946, symbol ucc2946:UCC2946
- C2: renamed from C?; value 1n5 -> 1n
- D6: renamed from D?; value LED -> GREEN LED
- R8: renamed from R?; value 1k -> 330
- U5: renamed from U?; value LTV-356T -> VO618A
- gave numbers to parts that had none: 18
Connections:
- net +5V: now also R5.1, C4.1, C5.1, R12.1, R9.1, SW1.6 (C), U4.8 (VDD); no longer R5.2
- net GND: now also C3.2, C4.2, C5.2, D1.1 (K), D2.1 (K), D5.1 (K), SW1.3 (C), U3.2, U4.1 (GND)
- net at R8.1: now also U3.1
- net WATCHDOGpin: now reaches U1.~ (WDI)
- net WATCHDOGpin: now also R5.2
- net at R8.2: now also SW1.2 (B)
- net at R2.2: now also D2.2 (A)
- net at D7.1 (K): now also SW3.1 (A)
- net NTCpin: now reaches R3.2, TH1.1
- net ONE_WIRE_BUS: now reaches R4.2, U2.2 (DQ)
- net SERVERFAILpin: now reaches R2.1
- net at R11.2, U5.4: now also U4.7 (WDI)
- net RESET: now reaches SW2.2 (B)
- net at C2.1: now also U4.4 (RP)
- removed net WDI: R5.1, U1.~ (WDI)
- new net: R12.2, SW3.3 (C), U4.5 (WDO)
- new net: R7.2, SW1.5 (B)
- new net: D5.2 (A), R7.1
- new net: R9.2, U4.2 (RTH)
- new net: C3.1, U4.6 (WP)
- new net: D1.2 (A), R1.2
- new net INTERLOCKpin: SW1.4 (A)
- new net RELAYpin: SW1.1 (A)
- new net TXONpin: R1.1
- new net USRPpin: SW3.2 (B)
- new net VIN+12V: U3.6
- new net VOUT+12V: U3.5
- no-connect marks 10 -> 6
Other:
- note added: "Disable USRP watchdog"
- note added: "Disable watchdog reset\n(needed for reprogramming Arduino)"
- note added: "Heartbeat from the USRP\n3V3 logic levels"
- note added: "Manual interlock switch - disable all transmissions"
- note added: "The reset period\nT_RP (ms) = 3.125 x C_RP (nF). \nNot relevant for this\ncircuit..."
- note added: "The watchdog period T_WP (ms) = 25 x C_WP (nF).\nSo, with C=330nF the period is a bit more than 8s."
- note added: "With C=470pF, the watchdog periods are roughly\n- 16 seconds after reset\n- 4 seconds after the first WDI change"
- note removed: "Arduino Ethernet"
- note removed: "Heartbeat from the USRP"
- note removed: "With C=1.5nF, the watchdog periods are roughly\n- 51 seconds after reset\n- 6 seconds afterwards\nNOTE: this is not a good watchdog for the USRP!"
- note removed: "With C=470pF, the watchdog periods are roughly\n- 16 seconds after reset\n- 4 seconds afterwards"
- moved on the sheet: C1, C2, D3, D4, D6, D7, J1, J2, R10, R11, R13, R2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

Commit message: Added voltage monitoring
Parts:
- added D?: GREEN LED, symbol Device:LED
- added R?: 820, symbol Device:R
- added R?: 33k, symbol Device:R
- added R?: 10k, symbol Device:R
- D3: value LED -> RED LED
- R5: value 33 -> 33k
Connections:
- net GND: now also D?.1 (K), R?.2
- net VOUT+12V: now also R?.1, R?.2
- net WDO: now reaches D3.1 (K), U1.14 (WDO)
- net DISABLE_USRP_INTERLOCK: now reaches D7.1 (K), SW3.1 (A)
- net at R12.2, SW3.3 (C): no longer U4.5 (WDO)
- net nRESET: now reaches D4.1 (K), SW2.1 (A)
- net INTERLOCK_ON: now reaches R7.2, SW1.5 (B)
- net TXONpin renamed TOGGLEpin
- new net: D?.2 (A), R?.1
- new net USRP_WDO: U4.5 (WDO)
- new net VMONpin: R?.1, R?.2
Other:
- note added: "Arduino A0"
- note added: "Arduino A1"
- note added: "Connection fail"
- note added: "Interlock alive"
- note added: "Interlock on"
- note added: "Measure the PA power supply voltage"
- note added: "PA power on"
- note added: "USRP alive"
- note added: "USRP watchdog bypass"
- note added: "Watchdog timeout"
- moved on the sheet: C1, C2, C3, C4, C5, D1, D2, D3, D4, D5, D6, D7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

Commit message: Small corrections
Parts:
- added U?: VO618A, Package_SO:SO-4_4.4x3.6mm_P2.54mm, symbol Isolator:LTV-356T
- R?: value 33k -> 4k7
- R?: value 10k -> ??
Connections:
- net labels added: GNDPWR
- wire segments 117 -> 123
- no-connect marks 6 -> 7
Other:
- note added: "Arduino RESET"
- note added: "Check whether the PA power supply\nis on or not"
- note added: "RF PA power switch\n("C" connection, see datasheet)"
- note removed: "Measure the PA power supply voltage"
- note removed: "RF PA power switch"
- moved on the sheet: R?
Changed lines of the file:
@@
 Wire Wire Line
 	1700 4600 1650 4600
-Text Notes 5300 5900 2    50   Italic 0
-RF PA power switch
+Text Notes 4850 6000 0    50   Italic 0
+RF PA power switch\n("C" connection, see datasheet)
 Text Notes 8750 4450 2    50   Italic 0
 Attached to RF PA heat sink
@@
 	3250 6300 3650 6300
 Wire Wire Line
-	5050 6300 5550 6300
+	5050 6300 5250 6300
 Text GLabel 5550 6300 2    50   Input ~ 0
 VIN+12V
@@
 $EndComp
 $Comp
-L power:GND #PWR?
-U 1 1 5ED7D7F1
-P 5900 2150
-F 0 "#PWR?" H 5900 1900 50  0001 C CNN
-F 1 "GND" H 5905 1977 50  0000 C CNN
-F 2 "" H 5900 2150 50  0001 C CNN
-F 3 "" H 5900 2150 50  0001 C CNN
-	1    5900 2150
-	1    0    0    -1
-$EndComp
-$Comp
 L Device:R R?
 U 1 1 5ED7DCA5
@@
 Wire Wire Line
 	5900 1750 5900 1700
-Wire Wire Line
-	5900 2150 5900 2050
 Text Notes 6150 2600 2    50   Italic 0
 PA power on
@@
 Wire Wire Line
 	1600 10400 1750 10400
-Wire Wire Line
-	2050 10400 2200 10400
 Text GLabel 13350 8150 2    50   Input Italic 0
 USRP_WDO
-Wire Wire Line
-	2100 10800 2200 10800
-Wire Wire Line
-	2200 10800 2200 10400
-Connection ~ 2200 10400
-Wire Wire Line
-	2200 10400 2400 10400
-Text GLabel 10300 3950 1    50   Input ~ 0
+Text GLabel 6100 8300 1    50   Input ~ 0
 VOUT+12V
 $Comp
 L Device:R R?
 U 1 1 5EDF7D7C
-P 10300 4250
-F 0 "R?" H 10370 4296 50  0000 L CNN
-F 1 "33k" H 10370 4205 50  0000 L CNN
-F 2 "" V 10230 4250 50  0001 C CNN
-F 3 "~" H 10300 4250 50  0001 C CNN
-	1    10300 4250
+P 6950 8650
+F 0 "R?" H 7020 8696 50  0000 L CNN
+F 1 "4k7" H 7020 8605 50  0000 L CNN
+F 2 "" V 6880 8650 50  0001 C CNN
+F 3 "~" H 6950 8650 50  0001 C CNN
+	1    6950 8650
 	1    0    0    -1
 $EndComp
@@
 L Device:R R?
 U 1 1 5EDF82B4
-P 10300 4750
-F 0 "R?" H 10370 4796 50  0000 L CNN
-F 1 "10k" H 10370 4705 50  0000 L CNN
-F 2 "" V 10230 4750 50  0001 C CNN
-F 3 "~" H 10300 4750 50  0001 C CNN
-	1    10300 4750
-	1    0    0    -1
-$EndComp
-$Comp
-L power:GND #PWR?
-U 1 1 5EDF861D
-P 10300 5000
-F 0 "#PWR?" H 10300 4750 50  0001 C CNN
-F 1 "GND" H 10305 4827 50  0000 C CNN
-F 2 "" H 10300 5000 50  0001 C CNN
-F 3 "" H 10300 5000 50  0001 C CNN
-	1    10300 5000
-	1    0    0    -1
-$EndComp
-Wire Wire Line
-	10300 5000 10300 4900
-Wire Wire Line
-	10300 4100 10300 3950
-Wire Wire Line
-	10300 4600 10300 4450
-Text GLabel 9950 4450 0    50   Input ~ 0
+P 6100 8600
+F 0 "R?" H 6170 8646 50  0000 L CNN
+F 1 "??" H 6170 8555 50  0000 L CNN
+F 2 "" V 6030 8600 50  0001 C CNN
+F 3 "~" H 6100 8600 50  0001 C CNN
+	1    6100 8600
+	1    0    0    -1
+$EndComp
+Text GLabel 7350 8850 2    50   Input ~ 0
 VMONpin
-Wire Wire Line
-	9950 4450 10300 4450
-Connection ~ 10300 4450
-Wire Wire Line
-	10300 4450 10300 4400
-Text Notes 9650 5350 0    50   ~ 0
-Measure the PA power supply voltage
+Text Notes 6150 9700 0    50   ~ 0
+Check whether the PA power supply\nis on or not
 Text Notes 6850 4300 0    50   ~ 0
 Arduino A0
-Text Notes 9550 4350 0    50   ~ 0
+Text Notes 7750 9000 2    50   ~ 0
 Arduino A1
 Text GLabel 3250 1200 1    50   Input ~ 0
 TOGGLEpin
+Wire Wire Line
+	5050 6800 5250 6800
+Wire Wire Line
+	5250 6800 5250 6300
+Connection ~ 5250 6300
+Wire Wire Line
+	5250 6300 5550 6300
+Wire Wire Line
+	2050 10400 2400 10400
+NoConn ~ 3650 6800
+Text Notes 3050 8300 0    50   ~ 0
+Arduino RESET
+$Comp
+L Isolator:LTV-356T U?
+U 1 1 5F7EE090
+P 6500 8950
+F 0 "U?" H 6500 9275 50  0000 C CNN
+F 1 "VO618A" H 6500 9184 50  0000 C CNN
+F 2 "Package_SO:SO-4_4.4x3.6mm_P2.54mm" H 6300 8750 50  0001 L CIN
+F 3 "http://optoelectronics.liteon.com/upload/download/DS70-2001-010/S_110_LTV-356T%2020140520.pdf" H 6500 8950 50  0001 L CNN
+	1    6500 8950
+	1    0    0    -1
+$EndComp
+$Comp
+L power:GNDPWR #PWR?
+U 1 1 5F7F014A
+P 6100 9200
+F 0 "#PWR?" H 6100 9000 50  0001 C CNN
+F 1 "GNDPWR" H 6104 9046 50  0000 C CNN
+F 2 "" H 6100 9150 50  0001 C CNN
+F 3 "" H 6100 9150 50  0001 C CNN
+	1    6100 9200
+	1    0    0    -1
+$EndComp
+$Comp
+L power:GNDPWR #PWR?
+U 1 1 5F7F1672
+P 5900 2250
+F 0 "#PWR?" H 5900 2050 50  0001 C CNN
+F 1 "GNDPWR" H 5904 2096 50  0000 C CNN
+F 2 "" H 5900 2200 50  0001 C CNN
+F 3 "" H 5900 2200 50  0001 C CNN
+	1    5900 2250
+	1    0    0    -1
+$EndComp
+Wire Wire Line
+	5900 2050 5900 2250
+Wire Wire Line
+	6100 8300 6100 8450
+Wire Wire Line
+	6100 8750 6100 8850
+Wire Wire Line
+	6100 8850 6200 8850
+Wire Wire Line
+	6200 9050 6100 9050
+Wire Wire Line
+	6100 9050 6100 9200
+$Comp
+L power:GND #PWR?
+U 1 1 5F803EDD
+P 6850 9150
+F 0 "#PWR?" H 6850 8900 50  0001 C CNN
+F 1 "GND" H 6855 8977 50  0000 C CNN
+F 2 "" H 6850 9150 50  0001 C CNN
+F 3 "" H 6850 9150 50  0001 C CNN
+	1    6850 9150
+	1    0    0    -1
+$EndComp
+Wire Wire Line
+	6800 9050 6850 9050
+Wire Wire Line
+	6850 9050 6850 9150
+$Comp
+L power:+5V #PWR?
+U 1 1 5F80E6CF
+P 6950 8450
+F 0 "#PWR?" H 6950 8300 50  0001 C CNN
+F 1 "+5V" H 6965 8623 50  0000 C CNN
+F 2 "" H 6950 8450 50  0001 C CNN
+F 3 "" H 6950 8450 50  0001 C CNN
+	1    6950 8450
+	-1   0    0    -1
+$EndComp
+Wire Wire Line
+	6950 8450 6950 8500
+Wire Wire Line
+	6800 8850 6950 8850
+Wire Wire Line
+	6950 8850 6950 8800
+Wire Wire Line
+	6950 8850 7350 8850
+Connection ~ 6950 8850
 $EndSCHEMATC
